File: homer_thalamus/homer_thalamus.kicad_pcb (KiCad board)
At the start: 2 copper layers, 65 x 56 mm, 5 parts, among them J1 GPIO

Commit message: update pcb setup and edge cut
Other:
- board size 65 x 56 mm -> 95 x 56 mm
- copper layers 2 -> 4
- board text removed: "CAMERA (OPTIONAL)"
- board text removed: "DISPLAY (OPTIONAL)"
- board text removed: "Extend PCB edge 0.5mm if using SMT header"
- board text removed: "PoE"
- board text removed: "RJ45"
- board text removed: "USB"
