File: homer_thalamus/homer_thalamus.kicad_pcb (KiCad board)
At the start: 4 copper layers, 95 x 56 mm, 24 parts, among them J1 GPIO, J2 MotDrv_Pow_Conn, J3 Right_Motor_Conn, J4 Left_Motor_Conn, J5 Spare_GP_Conn, J6 VBUS_Conn, SW1 SW_PULLDOWN, U1 DRV8874_CARRIER_RIGHT, U2 DRV8874_CARRIER_LEFT, U3 HC-SR04

Commit message: update pcb layout
Parts:
- removed ACC1: GY-521, GY-521:GY-521
- added U4: HiLetGo-GY-521, GY-521:HiLetGo-GY-521, F.Cu at (83.5, 72.0)
- moved U3 1.27 mm to (73.8, 72.0)
- moved R6 0.38 mm to (116.8, 90.8)
- moved R1 0.35 mm to (124.4, 97.1)
- moved R5 0.35 mm to (124.4, 93.9)
- moved J6 0.19 mm to (163.1, 86.0)
Routing:
- added copper zone on B.Cu, net GND
- added copper zone on F.Cu, net GND
