File: homer_thalamus/homer_thalamus.kicad_pcb (KiCad board)
At the start: 4 copper layers, 95 x 56 mm, 27 parts, among them J1 GPIO, J2 MotDrv_Pow_Conn, J3 Right_Motor_Conn, J4 Left_Motor_Conn, J5 Spare_GP_Conn, J6 VBUS_Conn, SW1 SW_PULLDOWN, U1 DRV8874_CARRIER_RIGHT, U2 DRV8874_CARRIER_LEFT, U3 HC-SR04, U4 HiLetGo-GY-521

Commit message: minor update pcb labels and new gerber
Parts:
- D1: value LED_RKGB -> BGKR
- U4: value HiLetGo-GY-521 -> GY-521
Other:
- board text added: "+5V"
- board text added: "+7.4V"
- board text added: "ECHO"
- board text added: "MOT_POW"
- board text added: "TRIG"
- board text added: "USB"
- board text removed: "+"
Changed lines of the file:
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@@
 		(tags "connector JST XH vertical")
 		(property "Reference" "J2"
-			(at -3.9 -2.3 0)
+			(at -3.9 -2.3 90)
 			(layer "F.SilkS")
 			(effects
@@
 			)
 		)
-		(property "Value" "LED_RKGB"
+		(property "Value" "BGKR"
 			(at 3.211 3.725 0)
 			(layer "F.SilkS")
@@
 				(font
 					(size 1 1)
-					(thickness 0.1)
+					(thickness 0.15)
 				)
 			)
 		)
-		(property "Value" "HiLetGo-GY-521"
+		(property "Value" "GY-521"
 			(at -1.21 -10.7 0)
 			(unlocked yes)
@@
 		)
 	)
+	(gr_text "MOT_POW"
+		(at 71.3 88.6 90)
+		(layer "F.SilkS")
+		(effects
+			(font
+				(size 1 1)
+				(thickness 0.15)
+			)
+		)
+	)
 	(gr_text "GND"
 		(at 87.6 48 270)
@@
 		)
 	)
-	(gr_text "+"
-		(at 77 91.8 0)
+	(gr_text "+7.4V"
+		(at 76.8 92.2 0)
 		(layer "F.SilkS")
 		(effects
@@
 	)
 	(gr_text "-"
-		(at 74.2 91.8 0)
+		(at 74.2 92.2 0)
 		(layer "F.SilkS")
 		(effects
@@
 		)
 	)
+	(gr_text "USB"
+		(at 162.7 70.4 270)
+		(layer "F.SilkS")
+		(effects
+			(font
+				(size 1 1)
+				(thickness 0.15)
+			)
+			(justify left bottom)
+		)
+	)
 	(gr_text "GND"
 		(at 157.5 57.933333 270)
@@
 		)
 	)
+	(gr_text "ECHO"
+		(at 75 73.9 0)
+		(layer "B.SilkS")
+		(effects
+			(font
+				(size 1 1)
+				(thickness 0.15)
+			)
+			(justify right bottom mirror)
+		)
+	)
+	(gr_text "GND"
+		(at 75 76.4 0)
+		(layer "B.SilkS")
+		(effects
+			(font
+				(size 1 1)
+				(thickness 0.15)
+			)
+			(justify right bottom mirror)
+		)
+	)
+	(gr_text "+5V"
+		(at 75 68.8 0)
+		(layer "B.SilkS")
+		(effects
+			(font
+				(size 1 1)
+				(thickness 0.15)
+			)
+			(justify right bottom mirror)
+		)
+	)
+	(gr_text "TRIG"
+		(at 75 71.4 0)
+		(layer "B.SilkS")
+		(effects
+			(font
+				(size 1 1)
+				(thickness 0.15)
+			)
+			(justify right bottom mirror)
+		)
+	)

Commit message: update footprints
Parts:
- added J2: PICO_5VOUT, Connector_PinHeader_2.54mm:PinHeader_1x02_P2.54mm_Vertical, F.Cu at (121.6, 23.8)
- added J6: PICO_POW, Connector_PinHeader_2.54mm:PinHeader_1x02_P2.54mm_Horizontal, F.Cu at (108.3, 23.8)
- added J7: BAT_OUT, Connector_JST:JST_XH_B2B-XH-A_1x02_P2.50mm_Vertical, F.Cu at (122.0, 32.0)
- added J8: BAT_IN, TerminalBlock:TerminalBlock_MaiXu_MX126-5.0-02P_1x02_P5.00mm, F.Cu at (73.8, 109.5)
- D1: value BGKR -> LED_RKGB
- J5: value Spare_GP_Conn -> Spare_GP
- U4: value GY-521 -> HiLetGo-GY-521
Connections:
- net /BLUE renamed Net-(A1-GPIO26_ADC0)
- net /GREEN renamed Net-(A1-GPIO27_ADC1)
- net /RED renamed Net-(A1-GPIO28_ADC2)
- A1 pad 39: unconnected-(A1-VSYS-Pad39) -> VSYS

Commit message: pcb layout in progress
Parts:
- U3: moved to B.Cu
- moved C1 73.3 mm to (193.2, 95.8)
- moved D1 59.2 mm to (188.7, 109.9)
- moved R1 59.2 mm to (179.0, 119.7)
- moved R2 59.2 mm to (198.2, 115.4)
- moved R3 59.2 mm to (195.0, 115.4)
- moved R4 59.2 mm to (191.9, 115.4)
- moved R5 59.2 mm to (179.0, 116.6)
- moved R6 59.2 mm to (171.4, 113.4)
- moved SW1 59.2 mm to (181.8, 115.2)
- moved J6 49.3 mm to (209.0, 104.0)
- moved J4 27.2 mm to (102.2, 65.5), turned to 180 degrees
- moved A1 20.0 mm to (159.0, 72.0)
- moved J5 20.0 mm to (160.2, 52.7)
- moved U1 19.8 mm to (129.1, 94.8)
- moved U2 19.8 mm to (129.1, 73.7)
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- renumbered J8 to J1, J7 to J2, J4 to J3, J3 to J4, J2 to J7, J1 to J8, U2 to U1, U1 to U2
Routing:
- net VBUS: track 163.4 -> 0.00 mm, vias 1 -> 0
- net 3V3(OUT): track 106.0 -> 0.00 mm
- net /TRIG: track 72.7 -> 0.00 mm
- net Net-(U3-ECHO): track 53.4 -> 0.00 mm, vias 1 -> 0
- net /I2C0_SDA: track 52.9 -> 0.00 mm, vias 1 -> 0
- net /I2C0_SCL: track 52.3 -> 0.00 mm, vias 1 -> 0
- net /SW_PD: track 49.6 -> 0.00 mm
- net VMOT: track 43.6 -> 0.00 mm
- net /ENCA_L: track 41.4 -> 0.00 mm
- net /ENCA_R: track 40.8 -> 0.00 mm
- net /ENCB_R: track 39.6 -> 0.00 mm
- net /ENCB_L: track 36.4 -> 0.00 mm
- net /OUT1_R: track 23.0 -> 0.00 mm
- net /OUT2_L: track 20.5 -> 0.00 mm
- net /OUT2_R: track 19.4 -> 0.00 mm
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- removed copper zone on B.Cu, net GND
- removed copper zone on F.Cu, net GND
Other:
- board size 95 x 56 mm -> 85 x 56 mm

Commit message: pcb layout in progress
Parts:
- removed ? (x2): , 
- removed the J2 at (75.2, 95.7)
- removed the J6 at (209.0, 104.0)
- moved J6 99.9 mm to (180.2, 93.1)
- moved J7 88.4 mm to (176.5, 93.1)
- moved R1 69.9 mm to (145.0, 58.8)
- moved R5 69.9 mm to (145.0, 55.6)
- moved R6 69.9 mm to (137.4, 52.4)
- moved J1 62.7 mm to (108.1, 57.0), turned to 180 degrees
- moved C1 56.9 mm to (149.5, 59.5)
- moved SW1 49.4 mm to (138.1, 92.2), turned to 90 degrees
- moved J2 36.8 mm to (151.4, 54.0)
- moved R2 33.4 mm to (173.4, 93.0)
- moved R3 33.4 mm to (170.2, 93.0)
- moved R4 33.4 mm to (167.0, 93.0)
- moved U3 29.7 mm to (103.5, 72.0)
- moved J3 26.8 mm to (109.7, 97.2)
- moved U4 23.8 mm to (107.1, 75.1)
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
Commit message: in progress, pcb layout
Parts:
- moved R1 57.9 mm to (170.1, 110.9)
- moved R5 57.9 mm to (170.1, 107.7)
- moved R6 57.9 mm to (162.5, 104.6)
- moved J2 36.4 mm to (115.0, 53.7)
- moved D1 22.3 mm to (161.5, 85.0), turned to -90 degrees
- moved SW1 22.2 mm to (151.0, 110.3)
- moved J3 20.3 mm to (130.0, 97.3)
- moved J4 9.34 mm to (123.3, 54.8)
- moved C1 3.87 mm to (148.5, 55.7)
- moved J5 3.17 mm to (160.0, 55.9)
- moved U2 3.16 mm to (131.2, 77.1)
- moved U4 3.15 mm to (107.0, 72.0)
- moved J1 1.88 mm to (108.2, 55.1)
- moved U1 1.75 mm to (131.2, 95.2)
- moved U3 1.50 mm to (102.0, 72.0)
Routing:
- added copper zone on B.Cu, net GND
- added copper zone on F.Cu, net GND
Changed lines of the file:
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@@
 	(footprint "Connector_JST:JST_XH_B2B-XH-A_1x02_P2.50mm_Vertical"
 		(layer "F.Cu")
-		(at 151.4 54.05)
+		(at 115 53.7)
 		(descr "JST XH series connector, B2B-XH-A (http://www.jst-mfg.com/product/pdf/eng/eXH.pdf), generated with kicad-footprint-generator")
 		(tags "connector JST XH vertical")
@@
 	)
 	(footprint "RaspberryPi_Pico_THT:RaspberryPi_Pico_THT"
+		(locked yes)
 		(layer "F.Cu")
 		(at 159 72 -90)
@@
 	(footprint "Button_Switch_THT:SW_PUSH_6mm"
 		(layer "F.Cu")
-		(at 138.1 92.25 90)
+		(at 151 110.3 90)
 		(descr "Generic 6mm SW tactile push button")
 		(tags "tact sw push 6mm")
@@
 	(footprint "Resistor_THT:R_Axial_DIN0207_L6.3mm_D2.5mm_P7.62mm_Horizontal"
 		(layer "F.Cu")
-		(at 137.355 52.4254)
+		(at 162.48 104.5504)
 		(descr "Resistor, Axial_DIN0207 series, Axial, Horizontal, pin pitch=7.62mm, 0.25W = 1/4W, length*diameter=6.3*2.5mm^2, http://cdn-reichelt.de/documents/datenblatt/B400/1_4W%23YAG.pdf")
 		(tags "Resistor Axial_DIN0207 series Axial Horizontal pin pitch 7.62mm 0.25W = 1/4W length 6.3mm diameter 2.5mm")
@@
 	(footprint "DRV8874_Carrier:DRV8874_Carrier"
 		(layer "F.Cu")
-		(at 131.195 73.92 180)
+		(at 131.195 77.08 180)
 		(property "Reference" "U2"
 			(at 16.365 17.801 0)
@@
 			(polygon
 				(pts
-					(xy 131.1804 73.9146) (xy 115.9804 73.9146) (xy 115.9804 56.1146) (xy 131.1804 56.1146)
+					(xy 131.1804 77.0746) (xy 115.9804 77.0746) (xy 115.9804 59.2746) (xy 131.1804 59.2746)
 				)
 			)
@@
 			(polygon
 				(pts
-					(xy 131.1804 73.9146) (xy 115.9804 73.9146) (xy 115.9804 56.1146) (xy 131.1804 56.1146)
+					(xy 131.1804 77.0746) (xy 115.9804 77.0746) (xy 115.9804 59.2746) (xy 131.1804 59.2746)
 				)
 			)
@@
 	(footprint "Resistor_THT:R_Axial_DIN0207_L6.3mm_D2.5mm_P7.62mm_Horizontal"
 		(layer "F.Cu")
-		(at 144.975 55.575 180)
+		(at 170.1 107.7 180)
 		(descr "Resistor, Axial_DIN0207 series, Axial, Horizontal, pin pitch=7.62mm, 0.25W = 1/4W, length*diameter=6.3*2.5mm^2, http://cdn-reichelt.de/documents/datenblatt/B400/1_4W%23YAG.pdf")
 		(tags "Resistor Axial_DIN0207 series Axial Horizontal pin pitch 7.62mm 0.25W = 1/4W length 6.3mm diameter 2.5mm")
@@
 	(footprint "Resistor_THT:R_Axial_DIN0207_L6.3mm_D2.5mm_P7.62mm_Horizontal"
 		(layer "F.Cu")
-		(at 144.975 58.75 180)
+		(at 170.1 110.875 180)
 		(descr "Resistor, Axial_DIN0207 series, Axial, Horizontal, pin pitch=7.62mm, 0.25W = 1/4W, length*diameter=6.3*2.5mm^2, http://cdn-reichelt.de/documents/datenblatt/B400/1_4W%23YAG.pdf")
 		(tags "Resistor Axial_DIN0207 series Axial Horizontal pin pitch 7.62mm 0.25W = 1/4W length 6.3mm diameter 2.5mm")
@@
 	(footprint "LED_THT:LED_D5.0mm-4_RGB_Wide_Pins"
 		(layer "F.Cu")
-		(at 183.675 87.675 180)
+		(at 161.5 85.023 -90)
 		(descr "LED, diameter 5.0mm, 4 pins, WP154A4, https://www.kingbright.com/attachments/file/psearch/000/00/00/L-154A4SUREQBFZGEW(Ver.11A).pdf")
 		(tags "LED diameter 5.0mm 2 pins diameter 5.0mm 3 pins diameter 5.0mm 4 pins RGB RGBLED")
 		(property "Reference" "D1"
-			(at 8.636 2.54 0)
+			(at 8.636 2.54 90)
 			(layer "F.SilkS")
 			(effects
@@
 		)
 		(property "Value" "LED_RKGB"
-			(at 3.211 3.725 0)
+			(at 3.211 3.725 90)
 			(layer "F.SilkS")
 			(effects
@@
 		)
 		(property "Datasheet" "~"
-			(at 0 0 180)
+			(at 0 0 270)
 			(unlocked yes)
 			(layer "F.Fab")
@@
 		)
 		(property "Description" "RGB LED, red/cathode/green/blue"
-			(at 0 0 180)
+			(at 0 0 270)
 			(unlocked yes)
 			(layer "F.Fab")
@@
 		)
 		(fp_line
-			(start 7.56 3.25)
-			(end 7.56 -3.25)
+			(start -1.08 3.25)
+			(end 7.56 3.25)
 			(stroke
 				(width 0.05)
@@
 		)
 		(fp_line
-			(start 7.56 -3.25)
-			(end -1.08 -3.25)
+			(start 7.56 3.25)
+			(end 7.56 -3.25)
 			(stroke
 				(width 0.05)
@@
 		)
 		(fp_line
-			(start -1.08 3.25)
-			(end 7.56 3.25)
+			(start -1.08 -3.25)
+			(end -1.08 3.25)
 			(stroke
 				(width 0.05)
@@
 		)
 		(fp_line
-			(start -1.08 -3.25)
-			(end -1.08 3.25)
+			(start 7.56 -3.25)
+			(end -1.08 -3.25)
 			(stroke
 				(width 0.05)
@@
 		)
 		(fp_text user "${REFERENCE}"
-			(at 3.8862 5.2578 0)
+			(at 3.8862 5.2578 90)
 			(layer "F.Fab")
 			(effects
@@
 		)
 		(pad "1" thru_hole rect
-			(at 0 0 180)
+			(at 0 0 270)
 			(size 1.8 1.8)
 			(drill 0.9)
@@
 		)
 		(pad "2" thru_hole circle
-			(at 2.159 0 180)
+			(at 2.159 0 270)
 			(size 1.8 1.8)
 			(drill 0.9)
@@
 		)
 		(pad "3" thru_hole circle
-			(at 4.318 0 180)
+			(at 4.318 0 270)
 			(size 1.8 1.8)
 			(drill 0.9)
@@
 		)
 		(pad "4" thru_hole circle
-			(at 6.477 0 180)
+			(at 6.477 0 270)
 			(size 1.8 1.8)
 			(drill 0.9)
@@
 	(footprint "DRV8874_Carrier:DRV8874_Carrier"
 		(layer "F.Cu")
-		(at 131.2573 93.4527 180)
+		(at 131.2073 95.2027 180)
 		(property "Reference" "U1"
 			(at 15.365 18.404 0)
@@
 			(polygon
 				(pts
-					(xy 131.2427 93.4473) (xy 116.0427 93.4473) (xy 116.0427 75.6473) (xy 131.2427 75.6473)
+					(xy 131.1927 95.1973) (xy 115.9927 95.1973) (xy 115.9927 77.3973) (xy 131.1927 77.3973)
 				)
 			)
@@
 			(polygon
 				(pts
-					(xy 131.2427 93.4473) (xy 116.0427 93.4473) (xy 116.0427 75.6473) (xy 131.2427 75.6473)
+					(xy 131.1927 95.1973) (xy 115.9927 95.1973) (xy 115.9927 77.3973) (xy 131.1927 77.3973)
 				)
 			)
@@
 	)
 	(footprint "GY-521:HiLetGo-GY-521"
+		(locked yes)
 		(layer "F.Cu")
-		(at 107.12 75.145 180)
+		(at 107 72 180)
 		(property "Reference" "U4"
-			(at 6.24 -10.975 0)
+			(at 5.8 -10.8 0)
 			(unlocked yes)
 			(layer "F.SilkS")
@@
 			(polygon
 				(pts
-					(xy 115.62 85.145) (xy 100.12 85.145) (xy 100.12 64.445) (xy 115.62 64.445)
+					(xy 115.5 82) (xy 100 82) (xy 100 61.3) (xy 115.5 61.3)
 				)
 			)
@@
 	(footprint "Connector_PinHeader_2.54mm:PinHeader_1x06_P2.54mm_Vertical"
 		(layer "F.Cu")
-		(at 109.725 97.225 90)
+		(at 129.9873 97.3 90)
 		(descr "Through hole straight pin header, 1x06, 2.54mm pitch, single row")
 		(tags "Through hole pin header THT 1x06 2.54mm single row")
@@
 	(footprint "TerminalBlock:TerminalBlock_MaiXu_MX126-5.0-02P_1x02_P5.00mm"
 		(layer "F.Cu")
-		(at 108.075 56.975 180)
+		(at 108.2 55.1 180)
 		(descr "terminal block MaiXu MX126-5.0-02P, 2 pins, pitch 5mm, size 10.5x7.8mm, drill diameter 1.3mm, pad diameter 2.8mm, https://www.lcsc.com/datasheet/lcsc_datasheet_2309150913_MAX-MX126-5-0-03P-GN01-Cu-S-A_C5188435.pdf, script-generated using https://gitlab.com/kicad/libraries/kicad-footprint-generator/-/tree/master/scripts/TerminalBlock_MaiXu")
 		(tags "THT terminal block MaiXu MX126-5.0-02P pitch 5mm size 10.5x7.8mm drill 1.3mm pad 2.8mm")
@@
 	(footprint "Connector_PinHeader_2.54mm:PinHeader_1x06_P2.54mm_Vertical"
 		(layer "F.Cu")
-		(at 114.275 52.575 90)
+		(at 123.35 54.8 90)
 		(descr "Through hole straight pin header, 1x06, 2.54mm pitch, single row")
 		(tags "Through hole pin header THT 1x06 2.54mm single row")
@@
 	(footprint "Capacitor_THT:C_Disc_D4.7mm_W2.5mm_P5.00mm"
 		(layer "F.Cu")
-		(at 149.475 59.45)
+		(at 148.5 55.7)
 		(descr "C, Disc series, Radial, pin pitch=5.00mm, diameter*width=4.7*2.5mm^2, Capacitor, http://www.vishay.com/docs/45233/krseries.pdf")
 		(tags "C Disc series Radial pin pitch 5.00mm diameter 4.7mm width 2.5mm Capacitor")
@@
 	(footprint "Connector_PinHeader_2.54mm:PinHeader_1x10_P2.54mm_Vertical"
 		(layer "F.Cu")
-		(at 160.22 52.731 90)
+		(at 160.04 55.9 90)
 		(descr "Through hole straight pin header, 1x10, 2.54mm pitch, single row")
 		(tags "Through hole pin header THT 1x10 2.54mm single row")
@@
 	)
 	(footprint "Connector_PinSocket_2.54mm:PinSocket_2x20_P2.54mm_Vertical"
+		(locked yes)
 		(layer "B.Cu")
 		(at 108.37 48.77 -90)
@@
 	(footprint "HC-SR04:XCVR_HC-SR04"
 		(layer "B.Cu")
-		(at 103.5 72 90)
+		(at 102 72 90)
 		(property "Reference" "U3"
 			(at 6.3 -0.21 0)
@@
 		)
 		(property "Value" "HC-SR04"
-			(at -0.0162 -1.6738 90)
+			(at -0.0162 1.9 90)
 			(layer "B.SilkS")
 			(effects
@@
 	)
 	(gr_text "GND"
-		(at 160.125 90.325 270)
+		(at 165.7 97.1 270)
 		(layer "F.SilkS")
 		(effects
@@
 	)
 	(gr_text "VBUS"
-		(at 162.8 90.325 270)
+		(at 168.9 96.5 270)
 		(layer "F.SilkS")
 		(effects
@@
 		)
 	)
+	(zone
+		(net 1)
+		(net_name "GND")
+		(layers "F.Cu" "B.Cu")
+		(hatch edge 0.5)
+		(connect_pads
+			(clearance 0)
+		)
+		(min_thickness 0.25)
+		(filled_areas_thickness no)
+		(fill yes
+			(thermal_gap 0.5)
+			(thermal_bridge_width 0.5)
+		)
+		(polygon
+			(pts
+				(xy 95 32.1) (xy 95.5 110.5) (xy 194.5 110.875) (xy 191.8 32.7) (xy 94.9 32.3)
+			)
+		)
+	)
